Commit message: Update gripper_demo.urdf

File: urdf/gripper_demo.urdf (robot description, URDF)
Before this commit: robot Gripper URDF, 3 links, 2 joints
Links:
- link base_gripper: geometry collision mesh filename=package://gripper_demo/meshes/base_gripper.STL; visual mesh filename=package://gripper_demo/meshes/base_gripper.STL
- link bottom_finger: geometry collision mesh filename=package://gripper_demo/meshes/bottom_finger.STL; visual mesh filename=package://gripper_demo/meshes/bottom_finger.STL
- link top_finger: geometry collision mesh filename=package://gripper_demo/meshes/top_finger.STL; visual mesh filename=package://gripper_demo/meshes/top_finger.STL
